File: controller/pendant.kicad_pcb (KiCad board)
At the start: 4 copper layers, 33.2 x 33.2 mm, 43 parts, among them J1 Conn_01x04_Socket, J2 Conn_01x04_Socket, J3 Conn_01x04_Socket, J4 USB_C_Receptacle_PowerOnly_6P, J5 Conn_01x02_Socket, Q1 BSS138W, Q2 BSS138W, U1 XC6206P332MR, U2 LIS3DHTR_C15134, U3 STM32C071G8U6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

Commit message: feat: journal, pcb, prod files
Connections:
- TP1 pad 1: /SWD -> /SWC
Routing:
- net /SWD: track 10.5 -> 4.34 mm
- net /SWC: track 3.15 -> 8.26 mm
Changed lines of the file:
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@@
 			)
 		)
+		(property "LCSC" "C18357552"
+			(at 0 0 90)
+			(unlocked yes)
+			(layer "F.Fab")
+			(hide yes)
+			(effects
+				(font
+					(size 1 1)
+					(thickness 0.15)
+				)
+			)
+		)
 		(property ki_fp_filters "USB*C*Receptacle*")
 		(sheetname "/")
@@
 			(size 1 1)
 			(layers "F.Cu" "F.Mask")
-			(net 20 "/SWD")
+			(net 21 "/SWC")
 			(pinfunction "1")
 			(pintype "passive")
@@
 			)
 		)
+		(property "LCSC" "C16581"
+			(at 0 0 180)
+			(unlocked yes)
+			(layer "F.Fab")
+			(hide yes)
+			(effects
+				(font
+					(size 1 1)
+					(thickness 0.15)
+				)
+			)
+		)
 		(property ki_fp_filters "*SO*3.9x4.*P1.27mm*EP2.4*x3.3*mm*")
 		(sheetname "/")
@@
 			)
 		)
+		(property "LCSC" "C915088"
+			(at 0 0 180)
+			(unlocked yes)
+			(layer "F.Fab")
+			(hide yes)
+			(effects
+				(font
+					(size 1 1)
+					(thickness 0.15)
+				)
+			)
+		)
 		(property ki_fp_filters "Texas*RWU0007A*VQFN*2x2mm*P0.5mm*")
 		(sheetname "/")
@@
 			)
 		)
+		(property "LCSC" "C22392482"
+			(at 0 0 90)
+			(unlocked yes)
+			(layer "F.Fab")
+			(hide yes)
+			(effects
+				(font
+					(size 1 1)
+					(thickness 0.15)
+				)
+			)
+		)
 		(property ki_fp_filters "SOT?323*")
 		(sheetname "/")
@@
 	)
 	(segment
-		(start 175.7 75.255001)
-		(end 175.7 79.75)
-		(width 0.2)
-		(layer "F.Cu")
-		(net 20)
-	)
-	(segment
 		(start 179.991919 74.801)
 		(end 180.66147 75.470551)
@@
 	)
 	(segment
-		(start 177.13 74.6)
-		(end 176.355001 74.6)
-		(width 0.2)
-		(layer "F.Cu")
-		(net 20)
-	)
-	(segment
-		(start 176.355001 74.6)
-		(end 175.7 75.255001)
+		(start 180.66147 75.470551)
+		(end 180.66147 75.92)
 		(width 0.2)
 		(layer "F.Cu")
@@
 	)
 	(segment
-		(start 180.66147 75.470551)
-		(end 180.66147 75.92)
+		(start 175.7 76.4)
+		(end 176.5 75.6)
 		(width 0.2)
 		(layer "F.Cu")
-		(net 20)
+		(net 21)
 	)
 	(segment
@@
 		(width 0.2)
 		(layer "F.Cu")
+		(net 21)
+	)
+	(segment
+		(start 175.7 79.75)
+		(end 175.7 76.4)
+		(width 0.2)
+		(layer "F.Cu")
+		(net 21)
+	)
+	(segment
+		(start 176.5 75.6)
+		(end 177.13 75.6)
+		(width 0.2)
+		(layer "F.Cu")

Commit message: feat: power fixes
Parts:
- removed U5: LM66200DRLR, easyeda2kicad:SOT-583-8_L2.1-W1.2-P0.50-LS1.6-BL
- added D3: SS34, PCM_JLCPCB:D_SMA, F.Cu at (197.4, 86.0)
- added Q3: BSS138W, Package_TO_SOT_SMD:SOT-323_SC-70, F.Cu at (190.2, 87.1)
- added R12: 10kΩ, PCM_JLCPCB:R_0402, F.Cu at (189.9, 84.8)
- added R13: 120Ω, PCM_JLCPCB:R_0402, F.Cu at (191.8, 84.8)
- R6: value 20kΩ -> 100kΩ
- moved R6 13.2 mm to (189.1, 91.0), turned to 90 degrees
Connections:
- C10 pad 1: VBUCK -> +5V
- C11 pad 1: VBUCK -> +5V
- R1 pad 1: VBUCK -> +5V
- R6 pad 1: VBUS -> +BATT
- R6 pad 2: Net-(U5-ST) -> /EN
- U4 pad 3: VBUCK -> +5V
- U4 pad 5: +BATT -> /EN
Routing:
- net /EN: track 0.00 -> 7.58 mm
- net +BATT: track 18.6 -> 11.3 mm
- net +5V: track 15.2 -> 9.48 mm
- net VBUS: track 62.6 -> 59.0 mm
- net Net-(U5-ST): track 3.58 -> 0.00 mm
- net Net-(Q3-G): track 0.00 -> 2.58 mm
- net VBUCK: track 1.65 -> 0.00 mm
- net GND: track 36.6 -> 36.1 mm, vias 38 -> 35
- added copper zone on F.Cu, net +5V
- removed copper zone on F.Cu, net VBUCK

Commit message: feat: other changes
Parts:
- removed U2: LIS3DHTR_C15134, easyeda2kicad:LGA-16_L3.0-W3.0-P0.50-TL
- added U5: LIS2DW12TR, easyeda2kicad:LGA-12_L2.0-W2.0-P0.50-BL, F.Cu at (186.4, 78.9)
- moved C4 4.47 mm to (187.9, 81.7)
- moved C7 0.91 mm to (185.8, 80.9)
- moved C8 0.91 mm to (185.8, 82.2)
Connections:
- C4 pad 1: +3V3 -> GND
- C4 pad 2: GND -> +3V3
Routing:
- net GND: track 36.1 -> 30.3 mm, vias 35 -> 34
- net +3V3: track 34.4 -> 30.6 mm
- net /MOSI: track 6.34 -> 2.97 mm
- net /SCK: track 8.05 -> 4.91 mm
- net /INT: track 3.15 -> 5.63 mm, vias 0 -> 2
- net /MISO: track 5.66 -> 3.37 mm, vias 0 -> 2
- net /CS: track 4.91 -> 4.39 mm, vias 2 -> 0
