File: controller/pendant.kicad_sch (KiCad schematic)
At the start: 43 parts, among them J1 Conn_01x04_Socket, J2 Conn_01x04_Socket, J3 Conn_01x04_Socket, J4 USB_C_Receptacle_PowerOnly_6P, J5 Conn_01x02_Socket, Q1 BSS138W, Q2 BSS138W, U1 XC6206P332MR, U2 LIS3DHTR_C15134, U3 STM32C071G8U6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

Commit message: feat: journal, pcb, prod files
Parts:
- D1: LCSC (none) -> C22392482
- J4: LCSC (none) -> C18357552
- U4: LCSC (none) -> C915088
- U6: LCSC (none) -> C16581
Connections:
- net SWC: now also TP1.1
- net SWD: no longer TP1.1
Other:
- moved on the sheet: TP1
Changed lines of the file:
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@@
 	)
 	(junction
-		(at 210.82 59.69)
+		(at 97.79 78.74)
 		(diameter 0)
 		(color 0 0 0 0)
 	)
 	(junction
-		(at 156.21 33.02)
+		(at 210.82 59.69)
 		(diameter 0)
 		(color 0 0 0 0)
 	)
 	(junction
-		(at 208.28 59.69)
+		(at 156.21 33.02)
 		(diameter 0)
 		(color 0 0 0 0)
 	)
 	(junction
-		(at 97.79 81.28)
+		(at 208.28 59.69)
 		(diameter 0)
 		(color 0 0 0 0)
@@
 	(wire
 		(pts
-			(xy 97.79 81.28) (xy 99.06 81.28)
-		)
-		(stroke
-			(width 0)
-			(type default)
-		)
-	)
-	(wire
-		(pts
 			(xy 67.31 66.04) (xy 68.58 66.04)
 		)
@@
 	(wire
 		(pts
+			(xy 105.41 74.93) (xy 97.79 74.93)
+		)
+		(stroke
+			(width 0)
+			(type default)
+		)
+	)
+	(wire
+		(pts
 			(xy 251.46 36.83) (xy 248.92 36.83)
 		)
@@
 	(wire
 		(pts
-			(xy 105.41 82.55) (xy 97.79 82.55)
-		)
-		(stroke
-			(width 0)
-			(type default)
-		)
-	)
-	(wire
-		(pts
 			(xy 38.1 137.16) (xy 53.34 137.16)
 		)
@@
 	(wire
 		(pts
-			(xy 96.52 81.28) (xy 97.79 81.28)
+			(xy 96.52 81.28) (xy 99.06 81.28)
 		)
 		(stroke
@@
 	(wire
 		(pts
-			(xy 96.52 78.74) (xy 99.06 78.74)
+			(xy 96.52 78.74) (xy 97.79 78.74)
 		)
 		(stroke
@@
 	(wire
 		(pts
-			(xy 97.79 82.55) (xy 97.79 81.28)
-		)
-		(stroke
-			(width 0)
-			(type default)
-		)
-	)
-	(wire
-		(pts
 			(xy 166.37 187.96) (xy 157.48 187.96)
 		)
@@
 	(wire
 		(pts
+			(xy 97.79 74.93) (xy 97.79 78.74)
+		)
+		(stroke
+			(width 0)
+			(type default)
+		)
+	)
+	(wire
+		(pts
 			(xy 265.43 113.03) (xy 262.89 113.03)
 		)
@@
 	(wire
 		(pts
+			(xy 97.79 78.74) (xy 99.06 78.74)
+		)
+		(stroke
+			(width 0)
+			(type default)
+		)
+	)
+	(wire
+		(pts
 			(xy 138.43 172.72) (xy 139.7 172.72)
 		)
@@
 	(symbol
 		(lib_id "Connector:TestPoint")
-		(at 105.41 82.55 270)
+		(at 105.41 74.93 270)
 		(unit 1)
 		(exclude_from_sim no)
@@
 		(fields_autoplaced yes)
 		(property "Reference" "TP1"
-			(at 110.49 81.2799 90)
+			(at 110.49 73.6599 90)
 			(effects
 				(font
@@
 		)
 		(property "Value" "TestPoint"
-			(at 110.49 83.8199 90)
+			(at 110.49 76.1999 90)
 			(effects
 				(font
@@
 		)
 		(property "Footprint" "TestPoint:TestPoint_Pad_D1.0mm"
-			(at 105.41 87.63 0)
+			(at 105.41 80.01 0)
 			(effects
 				(font
@@
 		)
 		(property "Datasheet" "~"
-			(at 105.41 87.63 0)
+			(at 105.41 80.01 0)
 			(effects
 				(font
@@
 		)
 		(property "Description" "test point"
-			(at 105.41 82.55 0)
+			(at 105.41 74.93 0)
 			(effects
 				(font
@@
 		)
 		(instances
-			(project ""
+			(project "pendant"
 				(path "/f7a02fd0-a6e9-40f1-b281-b8169eb64190"
 					(reference "TP1")
@@
 			)
 		)
+		(property "LCSC" "C16581"
+			(at 210.82 44.45 0)
+			(effects
+				(font
+					(size 1.27 1.27)
+				)
+				(hide yes)
+			)
+		)
 		(pin "5"
 		)
@@
 		(on_board yes)
 		(dnp no)
-		(fields_autoplaced yes)
 		(property "Reference" "U3"
-			(at 102.87 72.3198 0)
+			(at 91.694 66.548 0)
 			(effects
 				(font
@@
 		)
 		(property "Value" "STM32C071G8U6"
-			(at 102.87 74.8598 0)
+			(at 91.694 69.088 0)
 			(effects
 				(font
@@
 			)
 		)
+		(property "LCSC" "C915088"
+			(at 128.27 170.18 0)
+			(effects
+				(font
+					(size 1.27 1.27)
+				)
+				(hide yes)
+			)
+		)
 		(pin "2"
 		)
@@
 			)
 		)
+		(property "LCSC" "C22392482"
+			(at 30.48 121.92 0)
+			(effects
+				(font
+					(size 1.27 1.27)
+				)
+				(hide yes)
+			)
+		)
 		(pin "3"
 		)
@@
 			(at 238.76 105.41 0)
 			(effects
+				(font
+					(size 1.27 1.27)
+				)
+				(hide yes)
+			)
+		)
+		(property "LCSC" "C18357552"
+			(at 238.76 105.41 0)
+			(effects

Commit message: feat: power fixes
Parts:
- removed R6: 20kΩ, PCM_JLCPCB:R_0402, symbol PCM_JLCPCB-Resistors:0402,20kΩ
- removed U5: LM66200DRLR, easyeda2kicad:SOT-583-8_L2.1-W1.2-P0.50-LS1.6-BL, symbol easyeda2kicad:LM66200DRLR
- added D3: SS34, PCM_JLCPCB:D_SMA, symbol PCM_JLCPCB-Diodes:Schottky,SS34
- added Q3: BSS138W, Package_TO_SOT_SMD:SOT-323_SC-70, symbol PCM_JLCPCB-Transistors:NMOS,BSS138W
- added R12: 10kΩ, PCM_JLCPCB:R_0402, symbol PCM_JLCPCB-Resistors:0402,10kΩ
- added R13: 120Ω, PCM_JLCPCB:R_0402, symbol PCM_JLCPCB-Resistors:0402,120Ω
- added R6: 100kΩ, PCM_JLCPCB:R_0402, symbol PCM_JLCPCB-Resistors:0402,100kΩ
Connections:
- net VBUCK is gone; now on net +5V: C10.1, C11.1, R1.1, U4.3 (VOUT)
- net +5V: now also D3.1
- net +BATT: now also R6.1; no longer U4.5 (EN)
- net GND: now also Q3.2 (S), R12.2
- net VBUS: now also D3.2, R13.1
- new net: Q3.1 (G), R12.1, R13.2
- new net EN: Q3.3 (D), R6.2, U4.5 (EN)

Commit message: feat: other changes
Parts:
- removed U2: LIS3DHTR_C15134, easyeda2kicad:LGA-16_L3.0-W3.0-P0.50-TL, symbol easyeda2kicad:LIS3DHTR_C15134
- added U5: LIS2DW12TR, easyeda2kicad:LGA-12_L2.0-W2.0-P0.50-BL, symbol easyeda2kicad:LIS2DW12TR
Connections:
- net +3V3: now also C4.2, U5.10 (VDDIO), U5.9 (VDD); no longer C4.1
- net CS: now also U5.2 (CS)
- net GND: now also C4.1, U5.6 (GND), U5.7 (RES), U5.8 (GND); no longer C4.2
- net INT: now also U5.12 (INT1)
- net MISO: now also U5.3 (SDO/SA0)
- net MOSI: now also U5.4 (SDA/SDI/SDO)
- net SCK: now also U5.1 (SCL/SPC)
- no-connect marks 9 -> 5
Other:
- moved on the sheet: C4, C7, C8
